Commit message: Integrate operator interfaces and keep ROS running on faults
Restore the operator and vehicle interface update, add verified REMdevice CAN and generic USB input paths, and preserve diagnostics with latched ERROR handling for deployment faults. Include deployment integration, regression tests, manuals and commissioning documentation.

File: src/mobotic_description/urdf/moboterra.urdf.xacro (robot description, xacro)
@@ -94,3 +94,15 @@
   <xacro:module m="${p['modules'][2]}"/>
   <xacro:module m="${p['modules'][3]}"/>
+  <xacro:macro name="corner" params="c">
+    <link name="${c['name']}"/>
+    <joint name="${c['name']}_fixed" type="fixed">
+      <parent link="chassis"/><child link="${c['name']}"/>
+      <origin xyz="${c['xyz'][0]} ${c['xyz'][1]} ${c['xyz'][2]}" rpy="0 0 0"/>
+    </joint>
+  </xacro:macro>
+  <xacro:property name="corners" value="${p.get('reference_corners', [])}"/>
+  <xacro:if value="${len(corners) == 4}">
+    <xacro:corner c="${corners[0]}"/><xacro:corner c="${corners[1]}"/>
+    <xacro:corner c="${corners[2]}"/><xacro:corner c="${corners[3]}"/>
+  </xacro:if>
 </robot>

Commit message: Support two-module hardware STO and independent CAN bus rates
Select powered modules consistently across configuration, launch, URDF, and virtual checks. Allow the two-module Siemens hardware-STO chassis to start without PLC telemetry while retaining FlexiSoft requirements for four modules and the existing physical enable guards.

Read per-bus rates from the platform profile, fix Elmo TPDO configuration and scanner topic routing, and improve container health discovery and policy defaults. Add regression tests and setup documentation.

File: src/mobotic_description/urdf/moboterra.urdf.xacro (robot description, xacro)
@@ -54,5 +54,5 @@
   <xacro:scanner s="${p['scanners']['units'][0]}"/>
   <xacro:scanner s="${p['scanners']['units'][1]}"/>
-  <!-- Four powered modules, no casters. Fixed CAD mounts, geometry-free moving
+  <!-- Powered modules selected by the profile. Fixed CAD mounts, geometry-free moving
        steering frames, and floor-aligned tyre axes. Meshes are not recalibrated
        or resized when a custom platform profile is selected. -->
@@ -90,8 +90,11 @@
     </joint>
   </xacro:macro>
-  <xacro:module m="${p['modules'][0]}"/>
-  <xacro:module m="${p['modules'][1]}"/>
-  <xacro:module m="${p['modules'][2]}"/>
-  <xacro:module m="${p['modules'][3]}"/>
+  <xacro:macro name="selected_modules" params="items">
+    <xacro:if value="${len(items) > 0}">
+      <xacro:module m="${items[0]}"/>
+      <xacro:selected_modules items="${items[1:]}"/>
+    </xacro:if>
+  </xacro:macro>
+  <xacro:selected_modules items="${p['modules']}"/>
   <xacro:macro name="corner" params="c">
     <link name="${c['name']}"/>
